Commit message: feat：添加apriltag到world中

File: src/mid360_simulation/urdf/mid360_robot.xacro (robot description, xacro)
@@ -8,5 +8,5 @@
   <xacro:include filename="$(find mid360_simulation)/urdf/mid360.xacro"/>
  <!-- 导入Aprilag -->
-  <xacro:include filename="$(find mid360_simulation)/urdf/tag16h5_0.xacro"/>
+  <!-- <xacro:include filename="$(find mid360_simulation)/urdf/tag16h5_0.xacro"/> -->
   <!-- 机器人基础参数定义 - 正方形盒子 -->
   <xacro:property name="base_mass" value="2.0" />
@@ -54,22 +54,13 @@
     <origin xyz="0 0 ${base_height/2}" rpy="0 0 0"/>
   </joint>
-  <!-- 实例化修正版的 Mid-360 激光雷达 -->
-  <!-- 使用我们修正的版本，传递可视化参数 -->
-  <!-- <xacro:mid360_fixed
-    name="livox"
-    parent="base_link"
-    topic="livox"
-    laser_visualize="${laser_visualize}">
-    <origin xyz="0 0 0.15" rpy="0 0 0"/>
-  </xacro:mid360_fixed> -->
   <xacro:mid360 name="livox" parent="base_link" topic="mid360">
     <origin xyz="0 0 ${base_height/2 + 0.05}" rpy="0 0 0"/>
   </xacro:mid360>
   <!-- 将 AprilTag 阵列连接到机器人，避免多根链接错误 -->
-  <joint name="base_to_tag" type="fixed">
+  <!-- <joint name="base_to_tag" type="fixed">
     <parent link="base_link"/>
     <child link="tag16h5_0_link"/>
-    <origin xyz="${base_length/2 + 0.15} 0 0" rpy="0 0 0"/>
-  </joint>
+    <origin xyz="2 0 0.5" rpy="0 0 0"/>
+  </joint> -->
   <!-- Gazebo 材质定义 -->
   <gazebo reference="base_link">

File: src/mid360_simulation/urdf/tag16h5_0.xacro (robot description, xacro)
@@ -83,6 +83,6 @@
         <box size="${block_length} ${block_width} ${block_height}" />
       </geometry>
-      <material name="obstacle_red">
-        <color rgba="0.8 0.2 0.2 1" />  <!-- 深红色障碍物 -->
+      <material name="obstacle_white">
+        <color rgba="1.0 1.0 1.0 1" />  <!-- 白色障碍物 -->
       </material>
     </visual>
@@ -116,6 +116,6 @@
         <box size="${block_length} ${block_width} ${block_height}" />
       </geometry>
-      <material name="obstacle_red">
-        <color rgba="0.8 0.2 0.2 1" />
+      <material name="obstacle_white">
+        <color rgba="1.0 1.0 1.0 1" />
       </material>
     </visual>
@@ -146,6 +146,6 @@
         <box size="${block_length} ${block_width} ${block_height}" />
       </geometry>
-      <material name="obstacle_red">
-        <color rgba="0.8 0.2 0.2 1" />
+      <material name="obstacle_white">
+        <color rgba="1.0 1.0 1.0 1" />
       </material>
     </visual>
@@ -179,6 +179,6 @@
         <box size="${block_length} ${block_width} ${block_height}" />
       </geometry>
-      <material name="obstacle_red">
-        <color rgba="0.8 0.2 0.2 1" />
+      <material name="obstacle_white">
+        <color rgba="1.0 1.0 1.0 1" />
       </material>
     </visual>
@@ -212,6 +212,6 @@
         <box size="${block_length} ${block_width} ${block_height}" />
       </geometry>
-      <material name="obstacle_red">
-        <color rgba="0.8 0.2 0.2 1" />
+      <material name="obstacle_white">
+        <color rgba="1.0 1.0 1.0 1" />
       </material>
     </visual>
@@ -242,6 +242,6 @@
         <box size="${block_length} ${block_width} ${block_height}" />
       </geometry>
-      <material name="obstacle_red">
-        <color rgba="0.8 0.2 0.2 1" />
+      <material name="obstacle_white">
+        <color rgba="1.0 1.0 1.0 1" />
       </material>
     </visual>
@@ -272,6 +272,6 @@
         <box size="${block_length} ${block_width} ${block_height}" />
       </geometry>
-      <material name="obstacle_red">
-        <color rgba="0.8 0.2 0.2 1" />
+      <material name="obstacle_white">
+        <color rgba="1.0 1.0 1.0 1" />
       </material>
     </visual>
@@ -299,3 +299,32 @@
   <!-- 第6行 (i=5): [1 1 1 1 1 1] - 全部为1，无小长方体 -->
   <!-- =================================================================== -->
+  <!-- =================================================================== -->
+  <!-- Gazebo 材质定义 - 确保在 Gazebo 仿真中显示正确颜色 -->
+  <!-- =================================================================== -->
+  <!-- AprilTag 主体材质 -->
+  <gazebo reference="tag16h5_0_link">
+    <material>Gazebo/Purple</material>
+  </gazebo>
+  <!-- 小方块材质 - 白色 -->
+  <gazebo reference="block_1_3">
+    <material>Gazebo/White</material>
+  </gazebo>
+  <gazebo reference="block_2_3">
+    <material>Gazebo/White</material>
+  </gazebo>
+  <gazebo reference="block_2_4">
+    <material>Gazebo/White</material>
+  </gazebo>
+  <gazebo reference="block_3_4">
+    <material>Gazebo/White</material>
+  </gazebo>
+  <gazebo reference="block_4_1">
+    <material>Gazebo/White</material>
+  </gazebo>
+  <gazebo reference="block_4_3">
+    <material>Gazebo/White</material>
+  </gazebo>
+  <gazebo reference="block_4_4">
+    <material>Gazebo/White</material>
+  </gazebo>
 </robot>
